File: Processor1.sch (KiCad schematic (older format))
At the start: 13 parts, among them SW2 SW_PUSH, U3 AM3359AZCZ100, X1 24MHz, X2 CM200C

Commit message: Power supply
Connections:
- net labels added: DDR_VREF
Changed lines of the file:
@@
 LIBS:contrib
 LIBS:valves
+LIBS:gc
 LIBS:gc-cache
 EELAYER 24 0
@@
 	4200 9650 4200 9950
 Wire Wire Line
-	3400 8900 4800 8900
+	3370 8900 4800 8900
 Wire Wire Line
 	4200 9250 4200 8900
@@
 	4050 1850 4250 1850
 Connection ~ 3400 1850
+$Comp
+L DDR_VREF #PWR?
+U 1 1 5386EB1B
+P 3370 8900
+F 0 "#PWR?" H 3370 9040 20  0001 C CNN
+F 1 "DDR_VREF" H 3370 9010 30  0000 C CNN
+F 2 "" H 3370 8900 60  0000 C CNN
+F 3 "" H 3370 8900 60  0000 C CNN
+	1    3370 8900
+	0    -1   -1   0
+$EndComp
 $EndSCHEMATC
