File: gc.sch (KiCad schematic (older format))
At the start: 40 parts, among them J1 JACK_2P, P10 CONN_1, P11 CONN_1, P8 CONN_1, P9 CONN_1, SW1 SW_PUSH, U1 TL5209D, U2 TPC65217C

Commit message: Power supply
Connections:
- wire segments 141 -> 144
- no-connect marks 15 -> 14
Other:
- note added: "POWER_BUTTERY?\n"
Changed lines of the file:
@@
 LIBS:contrib
 LIBS:valves
+LIBS:gc
 LIBS:gc-cache
 EELAYER 24 0
@@
 $EndComp
 Wire Wire Line
-	2700 3050 2900 3050
-Wire Wire Line
 	5900 2700 5900 3550
 $Comp
@@
 $EndComp
 Wire Wire Line
-	2900 3050 2900 3400
-Wire Wire Line
 	3600 2650 3600 2900
-Wire Wire Line
-	2700 2800 3600 2800
-Connection ~ 3600 2800
 Wire Wire Line
 	3600 2700 5900 2700
@@
 	7500 3550 7700 3550
 Connection ~ 7700 3550
-NoConn ~ 2700 2950
 $Comp
 L CONN_1 P8
@@
 Text Notes 1515 2650 0    60   ~ 0
 POWER\n
+Wire Wire Line
+	2700 2800 2900 2800
+Wire Wire Line
+	2900 2800 2900 3400
+Wire Wire Line
+	2700 3050 3190 3050
+Wire Wire Line
+	3190 3050 3190 2795
+Wire Wire Line
+	3190 2795 3600 2795
+Connection ~ 3600 2795
+Wire Wire Line
+	2700 2950 2900 2950
+Connection ~ 2900 2950
+Text Notes 3660 4600 0    60   ~ 0
+POWER_BUTTERY?\n
 $EndSCHEMATC
